File: hardware/kicad/oso75/oso75.kicad_pcb (KiCad board)
At the start: 2 copper layers, 346.6 x 171.1 mm, 186 parts, among them J1 USB-C, SW1 MX_Hotswap, SW10 MX_Hotswap, SW11 MX_Hotswap, SW12 MX_Hotswap, SW13 MX_Hotswap, SW14 MX_Hotswap, SW15 MX_Hotswap, SW16 MX_Hotswap, SW17 MX_Hotswap, SW18 MX_Hotswap, SW19 MX_Hotswap, SW2 MX_Hotswap, SW20 MX_Hotswap, SW21 MX_Hotswap, SW22 MX_Hotswap, SW23 MX_Hotswap, SW24 MX_Hotswap, SW25 MX_Hotswap, SW26 MX_Hotswap, SW27 MX_Hotswap, SW28 MX_Hotswap, SW29 MX_Hotswap, SW3 MX_Hotswap, SW30 MX_Hotswap, SW31 MX_Hotswap, SW32 MX_Hotswap, SW33 MX_Hotswap, SW34 MX_Hotswap, SW35 MX_Hotswap, SW36 MX_Hotswap, SW37 MX_Hotswap, SW38 MX_Hotswap, SW39 MX_Hotswap, SW4 MX_Hotswap, SW40 MX_Hotswap, SW41 MX_Hotswap, SW42 MX_Hotswap, SW43 MX_Hotswap, SW44 MX_Hotswap, SW45 MX_Hotswap, SW46 MX_Hotswap, SW47 MX_Hotswap, SW48 MX_Hotswap, SW49 MX_Hotswap, SW5 MX_Hotswap, SW50 MX_Hotswap, SW51 MX_Hotswap, SW52 MX_Hotswap, SW53 MX_Hotswap, SW54 MX_Hotswap, SW55 MX_Hotswap, SW56 MX_Hotswap, SW57 MX_Hotswap, SW58 MX_Hotswap, SW59 MX_Hotswap, SW6 MX_Hotswap, SW60 MX_Hotswap, SW61 MX_Hotswap, SW62 MX_Hotswap, SW63 MX_Hotswap, SW64 MX_Hotswap, SW65 MX_Hotswap, SW66 MX_Hotswap, SW67 MX_Hotswap, SW68 MX_Hotswap, SW69 MX_Hotswap, SW7 MX_Hotswap, SW70 MX_Hotswap, SW71 MX_Hotswap, SW72 MX_Hotswap, SW73 MX_Hotswap, SW74 MX_Hotswap, SW75 MX_Hotswap, SW76 MX_Hotswap, SW77 MX_Hotswap, SW78 MX_Hotswap, SW79 MX_Hotswap, SW8 MX_Hotswap, SW80 MX_Hotswap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

Commit message: Update PCB for flush OSO module bay
Parts:
- removed D83, D84: 1N4148W, OSO75:D_SOD-123_Keyboard
- removed SW83, SW84: MX_Hotswap, OSO75:MX_Hotswap_1u
- added F1: 500mA, OSO75:Polyfuse_1206, F.Cu at (129.3, 134.1)
- added J3: OSO_Module_Bay_10, OSO75:OSO_Module_Bay_10, F.Cu at (38.0, 17.5)
- added R10: 10k, OSO75:R_0603, F.Cu at (140.3, 134.1)
- moved D13 248.8 mm to (44.1, 48.8)
- moved SW13 248.8 mm to (37.6, 42.3)
- moved D12 248.8 mm to (25.0, 48.8)
- moved SW12 248.8 mm to (18.5, 42.3)
- moved D40 231.8 mm to (32.2, 86.9)
- moved SW40 231.8 mm to (25.7, 80.4)
- moved D27 229.4 mm to (53.6, 67.9)
- moved SW27 229.4 mm to (47.1, 61.4)
- moved D41 229.4 mm to (58.4, 86.9)
- moved SW41 229.4 mm to (51.9, 80.4)
- moved D26 224.6 mm to (29.8, 67.9)
- moved SW26 224.6 mm to (23.3, 61.4)
- moved D66 215.2 mm to (51.2, 125.0)
- moved SW66 215.2 mm to (44.7, 118.5)
- moved D65 212.8 mm to (27.4, 125.0)
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Connections:
- D12 pad 2: ROW0 -> ROW1
- D13 pad 2: ROW0 -> ROW1
- D26 pad 2: ROW1 -> ROW2
- D27 pad 2: ROW1 -> ROW2
- D40 pad 2: ROW2 -> ROW3
- D41 pad 2: ROW2 -> ROW3
- D53 pad 2: ROW3 -> ROW4
- D54 pad 2: ROW3 -> ROW4
- D65 pad 2: ROW4 -> ROW5
- D66 pad 2: ROW4 -> ROW5
- D72 pad 2: ROW5 -> ROW0
- D73 pad 2: ROW5 -> ROW1
- D74 pad 2: ROW0 -> ROW1
- D75 pad 2: ROW1 -> ROW2
- D76 pad 2: ROW1 -> ROW2
- D77 pad 2: ROW2 -> ROW3
- D78 pad 2: ROW2 -> ROW3
- D79 pad 2: ROW3 -> ROW4
- D80 pad 2: ROW3 -> ROW5
- D81 pad 2: ROW4 -> ROW5
- SW1 pad 1: COL0 -> COL2
- SW10 pad 1: COL9 -> COL11
- SW11 pad 1: COL10 -> COL12
- SW12 pad 1: COL11 -> COL0
- SW13 pad 1: COL12 -> COL1
- SW14 pad 1: COL0 -> COL2
- SW15 pad 1: COL1 -> COL3
- SW16 pad 1: COL2 -> COL4
- SW17 pad 1: COL3 -> COL5
- SW18 pad 1: COL4 -> COL6
- SW19 pad 1: COL5 -> COL7
- SW2 pad 1: COL1 -> COL3
- SW20 pad 1: COL6 -> COL8
- SW21 pad 1: COL7 -> COL9
- SW22 pad 1: COL8 -> COL10
- SW23 pad 1: COL9 -> COL11
- SW24 pad 1: COL10 -> COL12
- SW25 pad 1: COL11 -> COL13
- SW26 pad 1: COL12 -> COL0
- SW27 pad 1: COL13 -> COL1
- SW28 pad 1: COL0 -> COL2
- SW29 pad 1: COL1 -> COL3
- SW3 pad 1: COL2 -> COL4
- SW30 pad 1: COL2 -> COL4
- SW31 pad 1: COL3 -> COL5
- SW32 pad 1: COL4 -> COL6
- SW33 pad 1: COL5 -> COL7
- SW34 pad 1: COL6 -> COL8
- SW35 pad 1: COL7 -> COL9
- SW36 pad 1: COL8 -> COL10
- SW37 pad 1: COL9 -> COL11
- SW38 pad 1: COL10 -> COL12
- SW39 pad 1: COL11 -> COL13
- SW4 pad 1: COL3 -> COL5
- SW40 pad 1: COL12 -> COL0
- SW41 pad 1: COL13 -> COL1
- SW42 pad 1: COL0 -> COL2
- SW43 pad 1: COL1 -> COL3
- SW44 pad 1: COL2 -> COL4
- SW45 pad 1: COL3 -> COL5
- SW46 pad 1: COL4 -> COL6
- SW47 pad 1: COL5 -> COL7
- SW48 pad 1: COL6 -> COL8
- SW49 pad 1: COL7 -> COL9
- SW5 pad 1: COL4 -> COL6
- SW50 pad 1: COL8 -> COL10
- SW51 pad 1: COL9 -> COL11
- SW52 pad 1: COL10 -> COL12
- SW53 pad 1: COL11 -> COL0
- SW54 pad 1: COL12 -> COL1
- SW55 pad 1: COL0 -> COL2
- SW56 pad 1: COL1 -> COL3
- SW57 pad 1: COL2 -> COL4
- SW58 pad 1: COL3 -> COL5
- SW59 pad 1: COL4 -> COL6
- SW6 pad 1: COL5 -> COL7
- SW60 pad 1: COL5 -> COL7
- SW61 pad 1: COL6 -> COL8
- SW62 pad 1: COL7 -> COL9
- SW63 pad 1: COL8 -> COL10
- SW64 pad 1: COL9 -> COL11
- SW65 pad 1: COL10 -> COL0
- SW66 pad 1: COL11 -> COL1
- SW67 pad 1: COL0 -> COL2
- SW68 pad 1: COL1 -> COL3
- SW69 pad 1: COL2 -> COL4
- SW7 pad 1: COL6 -> COL8
- SW70 pad 1: COL3 -> COL5
- SW71 pad 1: COL4 -> COL6
- SW72 pad 1: COL5 -> COL13
- SW73 pad 1: COL6 -> COL14
- SW74 pad 1: COL13 -> COL15
- SW77 pad 1: COL14 -> COL13
- SW78 pad 1: COL15 -> COL14
- SW79 pad 1: COL13 -> COL12
- SW8 pad 1: COL7 -> COL9
- SW80 pad 1: COL14 -> COL7
- SW81 pad 1: COL12 -> COL8
- SW82 pad 1: COL7 -> COL9
- SW9 pad 1: COL8 -> COL10
- U1 pad 37: GND -> MOD_INT
- U1 pad 38: ENC_A -> MOD_A
- U1 pad 39: ENC_B -> MOD_B
Routing:
- net D84_A: track 6.50 -> 0.00 mm
- net D83_A: track 6.50 -> 0.00 mm
Other:
- board size 346.6 x 171.1 mm -> 346.6 x 137.1 mm
