File: hardware/kicad/oso75/oso75.kicad_pcb (KiCad board)
At the start: 2 copper layers, 346.6 x 137.1 mm, 185 parts, among them J1 USB-C, J3 OSO_Module_Bay_10, SW1 MX_Hotswap, SW10 MX_Hotswap, SW11 MX_Hotswap, SW12 MX_Hotswap, SW13 MX_Hotswap, SW14 MX_Hotswap, SW15 MX_Hotswap, SW16 MX_Hotswap, SW17 MX_Hotswap, SW18 MX_Hotswap, SW19 MX_Hotswap, SW2 MX_Hotswap, SW20 MX_Hotswap, SW21 MX_Hotswap, SW22 MX_Hotswap, SW23 MX_Hotswap, SW24 MX_Hotswap, SW25 MX_Hotswap, SW26 MX_Hotswap, SW27 MX_Hotswap, SW28 MX_Hotswap, SW29 MX_Hotswap, SW3 MX_Hotswap, SW30 MX_Hotswap, SW31 MX_Hotswap, SW32 MX_Hotswap, SW33 MX_Hotswap, SW34 MX_Hotswap, SW35 MX_Hotswap, SW36 MX_Hotswap, SW37 MX_Hotswap, SW38 MX_Hotswap, SW39 MX_Hotswap, SW4 MX_Hotswap, SW40 MX_Hotswap, SW41 MX_Hotswap, SW42 MX_Hotswap, SW43 MX_Hotswap, SW44 MX_Hotswap, SW45 MX_Hotswap, SW46 MX_Hotswap, SW47 MX_Hotswap, SW48 MX_Hotswap, SW49 MX_Hotswap, SW5 MX_Hotswap, SW50 MX_Hotswap, SW51 MX_Hotswap, SW52 MX_Hotswap, SW53 MX_Hotswap, SW54 MX_Hotswap, SW55 MX_Hotswap, SW56 MX_Hotswap, SW57 MX_Hotswap, SW58 MX_Hotswap, SW59 MX_Hotswap, SW6 MX_Hotswap, SW60 MX_Hotswap, SW61 MX_Hotswap, SW62 MX_Hotswap, SW63 MX_Hotswap, SW64 MX_Hotswap, SW65 MX_Hotswap, SW66 MX_Hotswap, SW67 MX_Hotswap, SW68 MX_Hotswap, SW69 MX_Hotswap, SW7 MX_Hotswap, SW70 MX_Hotswap, SW71 MX_Hotswap, SW72 MX_Hotswap, SW73 MX_Hotswap, SW74 MX_Hotswap, SW75 MX_Hotswap, SW76 MX_Hotswap, SW77 MX_Hotswap, SW78 MX_Hotswap, SW79 MX_Hotswap, SW8 MX_Hotswap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

Commit message: Prepare OSO75 hardware review package
Parts:
- removed C5, C6: 18pF, OSO75:C_0603
- removed U2: W25Q128, Package_SO:SOIC-8_3.9x4.9mm_P1.27mm
- added C_EN: 1uF, OSO75:C_0603, F.Cu at (92.6, 9.06)
- added ST1: Stabilizer_Cherry_MX_2.00u, OSO75:Stabilizer_Cherry_MX_2.00u, F.Cu at (275.7, 55.3)
- added ST2: Stabilizer_Cherry_MX_2.00u, OSO75:Stabilizer_Cherry_MX_2.00u, F.Cu at (273.3, 93.4)
- added ST3: Stabilizer_Cherry_MX_2.00u, OSO75:Stabilizer_Cherry_MX_2.00u, F.Cu at (30.4, 112.5)
- added ST4: Stabilizer_Cherry_MX_6.25u, OSO75:Stabilizer_Cherry_MX_6.25u, F.Cu at (140.0, 131.5)
- C3: value 1uF -> 100nF
- F1: value 500mA -> 0603L050SLYR; footprint OSO75:Polyfuse_1206 -> OSO75:Polyfuse_0603
- J1: value USB-C -> USB_C_HRO_TYPE-C-31-M-12; footprint Connector_USB:USB_C_Receptacle_HRO_TYPE-C-31-M-12 -> OSO75:USB_C_Receptacle_HRO_TYPE-C-31-M-12
- J3: value OSO_Module_Bay_10 -> Exposed_OSO_Bay_Pads_DNP
- R5, R6: value 100k -> 10k
- SW1, SW10, SW11, SW12, SW13, SW14, SW15, SW16, SW17, SW18, SW19, SW2, SW20, SW21, SW22, SW23, SW24, SW25, SW26, SW27, SW28, SW29, SW3, SW30, SW31, SW32, SW33, SW34, SW35, SW36, SW37, SW38, SW39, SW4, SW40, SW41, SW42, SW43, SW44, SW45, SW46, SW47, SW48, SW49, SW5, SW50, SW51, SW52, SW53, SW54, SW55, SW56, SW57, SW58, SW59, SW6, SW60, SW61, SW62, SW63, SW64, SW65, SW66, SW67, SW68, SW69, SW7, SW70, SW71, SW72, SW73, SW74, SW75, SW76, SW77, SW78, SW79, SW8, SW80, SW81, SW82, SW9: footprint OSO75:MX_Hotswap_1u -> OSO75:SW_Hotswap_Kailh_MX_Plated_1.00u_With_Switch
- U1: value RP2040 -> ESP32-S3-WROOM-1U-N16; footprint Package_DFN_QFN:QFN-56-1EP_7x7mm_P0.4mm_EP4x4mm -> OSO75:ESP32-S3-WROOM-1U-N16
- moved SW_BOOT 156.3 mm to (101.5, 12.1), turned to 180 degrees
- moved J1 131.9 mm to (168.5, 2.40), turned to 180 degrees
- moved R6 127.8 mm to (131.5, 12.1), turned to 180 degrees
- moved R1 126.8 mm to (179.5, 3.06), turned to 180 degrees
- moved R10 125.8 mm to (109.5, 12.1), turned to 180 degrees
- moved SW_RESET 123.8 mm to (93.5, 12.1), turned to 180 degrees
- moved R2 123.0 mm to (179.5, 6.06), turned to 180 degrees
- moved F1 122.6 mm to (117.0, 12.1), turned to 180 degrees
- moved U3 121.8 mm to (147.0, 5.56), turned to 180 degrees
- moved C1 119.5 mm to (152.5, 5.56), turned to 180 degrees
- moved R3 119.5 mm to (157.5, 5.06), turned to 180 degrees
- moved U1 118.0 mm to (196.0, 11.3), turned to 90 degrees
- moved R4 117.4 mm to (157.5, 8.56), turned to 180 degrees
- moved C2 116.8 mm to (141.5, 5.56), turned to 180 degrees
- moved C4 114.5 mm to (181.0, 7.56), turned to 180 degrees
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Connections:
- C3 pad 1: +1V1 -> +3V3
- D1 pad 1: D1_A -> ROW0
- D1 pad 2: ROW0 -> D1_A
- D10 pad 1: D10_A -> ROW0
- D10 pad 2: ROW0 -> D10_A
- D11 pad 1: D11_A -> ROW0
- D11 pad 2: ROW0 -> D11_A
- D12 pad 1: D12_A -> ROW1
- D12 pad 2: ROW1 -> D12_A
- D13 pad 1: D13_A -> ROW1
- D13 pad 2: ROW1 -> D13_A
- D14 pad 1: D14_A -> ROW1
- D14 pad 2: ROW1 -> D14_A
- D15 pad 1: D15_A -> ROW1
- D15 pad 2: ROW1 -> D15_A
- D16 pad 1: D16_A -> ROW1
- D16 pad 2: ROW1 -> D16_A
- D17 pad 1: D17_A -> ROW1
- D17 pad 2: ROW1 -> D17_A
- D18 pad 1: D18_A -> ROW1
- D18 pad 2: ROW1 -> D18_A
- D19 pad 1: D19_A -> ROW1
- D19 pad 2: ROW1 -> D19_A
- D2 pad 1: D2_A -> ROW0
- D2 pad 2: ROW0 -> D2_A
- D20 pad 1: D20_A -> ROW1
- D20 pad 2: ROW1 -> D20_A
- D21 pad 1: D21_A -> ROW1
- D21 pad 2: ROW1 -> D21_A
- D22 pad 1: D22_A -> ROW1
- D22 pad 2: ROW1 -> D22_A
- D23 pad 1: D23_A -> ROW1
- D23 pad 2: ROW1 -> D23_A
- D24 pad 1: D24_A -> ROW1
- D24 pad 2: ROW1 -> D24_A
- D25 pad 1: D25_A -> ROW1
- D25 pad 2: ROW1 -> D25_A
- D26 pad 1: D26_A -> ROW2
- D26 pad 2: ROW2 -> D26_A
- D27 pad 1: D27_A -> ROW2
- D27 pad 2: ROW2 -> D27_A
- D28 pad 1: D28_A -> ROW2
- D28 pad 2: ROW2 -> D28_A
- D29 pad 1: D29_A -> ROW2
- D29 pad 2: ROW2 -> D29_A
- D3 pad 1: D3_A -> ROW0
- D3 pad 2: ROW0 -> D3_A
- D30 pad 1: D30_A -> ROW2
- D30 pad 2: ROW2 -> D30_A
- D31 pad 1: D31_A -> ROW2
- D31 pad 2: ROW2 -> D31_A
- D32 pad 1: D32_A -> ROW2
- D32 pad 2: ROW2 -> D32_A
- D33 pad 1: D33_A -> ROW2
- D33 pad 2: ROW2 -> D33_A
- D34 pad 1: D34_A -> ROW2
- D34 pad 2: ROW2 -> D34_A
- D35 pad 1: D35_A -> ROW2
- D35 pad 2: ROW2 -> D35_A
- D36 pad 1: D36_A -> ROW2
- D36 pad 2: ROW2 -> D36_A
- D37 pad 1: D37_A -> ROW2
- D37 pad 2: ROW2 -> D37_A
- D38 pad 1: D38_A -> ROW2
- D38 pad 2: ROW2 -> D38_A
- D39 pad 1: D39_A -> ROW2
- D39 pad 2: ROW2 -> D39_A
- D4 pad 1: D4_A -> ROW0
- D4 pad 2: ROW0 -> D4_A
- D40 pad 1: D40_A -> ROW3
- D40 pad 2: ROW3 -> D40_A
- D41 pad 1: D41_A -> ROW3
- D41 pad 2: ROW3 -> D41_A
- D42 pad 1: D42_A -> ROW3
- D42 pad 2: ROW3 -> D42_A
- D43 pad 1: D43_A -> ROW3
- D43 pad 2: ROW3 -> D43_A
- D44 pad 1: D44_A -> ROW3
- D44 pad 2: ROW3 -> D44_A
- D45 pad 1: D45_A -> ROW3
- D45 pad 2: ROW3 -> D45_A
- D46 pad 1: D46_A -> ROW3
- D46 pad 2: ROW3 -> D46_A
- D47 pad 1: D47_A -> ROW3
- D47 pad 2: ROW3 -> D47_A
- D48 pad 1: D48_A -> ROW3
- D48 pad 2: ROW3 -> D48_A
- D49 pad 1: D49_A -> ROW3
- D49 pad 2: ROW3 -> D49_A
- D5 pad 1: D5_A -> ROW0
- D5 pad 2: ROW0 -> D5_A
- D50 pad 1: D50_A -> ROW3
- D50 pad 2: ROW3 -> D50_A
- D51 pad 1: D51_A -> ROW3
- D51 pad 2: ROW3 -> D51_A
- D52 pad 1: D52_A -> ROW3
- D52 pad 2: ROW3 -> D52_A
- D53 pad 1: D53_A -> ROW4
- D53 pad 2: ROW4 -> D53_A
- D54 pad 1: D54_A -> ROW4
- D54 pad 2: ROW4 -> D54_A
- D55 pad 1: D55_A -> ROW4
- D55 pad 2: ROW4 -> D55_A
- D56 pad 1: D56_A -> ROW4
- D56 pad 2: ROW4 -> D56_A
- D57 pad 1: D57_A -> ROW4
- D57 pad 2: ROW4 -> D57_A
- D58 pad 1: D58_A -> ROW4
- D58 pad 2: ROW4 -> D58_A
- D59 pad 1: D59_A -> ROW4
- D59 pad 2: ROW4 -> D59_A
- D6 pad 1: D6_A -> ROW0
- D6 pad 2: ROW0 -> D6_A
- D60 pad 1: D60_A -> ROW4
- D60 pad 2: ROW4 -> D60_A
- D61 pad 1: D61_A -> ROW4
- D61 pad 2: ROW4 -> D61_A
- D62 pad 1: D62_A -> ROW4
- D62 pad 2: ROW4 -> D62_A
- D63 pad 1: D63_A -> ROW4
- D63 pad 2: ROW4 -> D63_A
- D64 pad 1: D64_A -> ROW4
- D64 pad 2: ROW4 -> D64_A
- D65 pad 1: D65_A -> ROW5
- D65 pad 2: ROW5 -> D65_A
- D66 pad 1: D66_A -> ROW5
- D66 pad 2: ROW5 -> D66_A
- D67 pad 1: D67_A -> ROW5
- D67 pad 2: ROW5 -> D67_A
- D68 pad 1: D68_A -> ROW5
- D68 pad 2: ROW5 -> D68_A
- D69 pad 1: D69_A -> ROW5
- D69 pad 2: ROW5 -> D69_A
- D7 pad 1: D7_A -> ROW0
- D7 pad 2: ROW0 -> D7_A
- D70 pad 1: D70_A -> ROW5
- D70 pad 2: ROW5 -> D70_A
- D71 pad 1: D71_A -> ROW5
- D71 pad 2: ROW5 -> D71_A
- D72 pad 1: D72_A -> ROW0
- D72 pad 2: ROW0 -> D72_A
- D73 pad 1: D73_A -> ROW1
- D73 pad 2: ROW1 -> D73_A
- D74 pad 1: D74_A -> ROW1
- D74 pad 2: ROW1 -> D74_A
- D75 pad 1: D75_A -> ROW2
- D75 pad 2: ROW2 -> D75_A
- D76 pad 1: D76_A -> ROW2
- D76 pad 2: ROW2 -> D76_A
- D77 pad 1: D77_A -> ROW3
- D77 pad 2: ROW3 -> D77_A
- D78 pad 1: D78_A -> ROW3
- D78 pad 2: ROW3 -> D78_A
- D79 pad 1: D79_A -> ROW4
- D79 pad 2: ROW4 -> D79_A
- D8 pad 1: D8_A -> ROW0
- D8 pad 2: ROW0 -> D8_A
- D80 pad 1: D80_A -> ROW5
- D80 pad 2: ROW5 -> D80_A
- D81 pad 1: D81_A -> ROW5
- D81 pad 2: ROW5 -> D81_A
- D82 pad 1: D82_A -> ROW5
- D82 pad 2: ROW5 -> D82_A
- D9 pad 1: D9_A -> ROW0
- D9 pad 2: ROW0 -> D9_A
- J3 pad 9: RESET_N -> ESP_EN
- R5 pad 1: RESET_N -> ESP_EN
- R6 pad 1: FLASH_CS_N -> BOOT_IO0
- SW68 pad 1: COL3 -> COL6
- SW69 pad 1: COL4 -> COL9
- SW70 pad 1: COL5 -> COL10
- SW71 pad 1: COL6 -> COL11
- SW77 pad 1: COL13 -> COL14
- SW78 pad 1: COL14 -> COL15
- SW79 pad 1: COL12 -> COL14
- SW80 pad 1: COL7 -> COL13
- SW81 pad 1: COL8 -> COL14
- SW82 pad 1: COL9 -> COL15
- SW_BOOT pad 1: FLASH_CS_N -> BOOT_IO0
- SW_RESET pad 1: RESET_N -> ESP_EN
- U1 pad 1: +3V3 -> GND
- U1 pad 10: +3V3 -> COL9
- U1 pad 11: COL2 -> COL10
- U1 pad 12: COL3 -> COL0
- U1 pad 13: COL4 -> USB_DM
- U1 pad 14: COL5 -> USB_DP
- U1 pad 15: COL6 -> (no net)
- U1 pad 16: COL7 -> (no net)
- U1 pad 17: COL8 -> COL1
- U1 pad 18: COL9 -> COL2
- U1 pad 19: GND -> COL3
- U1 pad 2: ROW0 -> +3V3
- U1 pad 20: XTAL_IN -> COL4
- U1 pad 21: XTAL_OUT -> COL5
- U1 pad 22: +3V3 -> COL6
- U1 pad 23: +1V1 -> COL11
- U1 pad 24: SWCLK -> MOD_INT
- U1 pad 25: SWDIO -> (no net)
- U1 pad 26: RESET_N -> (no net)
- U1 pad 27: COL10 -> BOOT_IO0
- U1 pad 28: COL11 -> COL12
- U1 pad 29: COL12 -> COL13
- U1 pad 3: ROW1 -> ESP_EN
- U1 pad 30: COL13 -> COL14
- U1 pad 31: COL14 -> COL15
- U1 pad 32: COL15 -> MOD_A
- U1 pad 33: +3V3 -> MOD_B
- U1 pad 34: LED_STATUS -> I2C_SDA
- U1 pad 35: GND -> I2C_SCL
- U1 pad 36: VBUS_SENSE -> (no net)
- U1 pad 37: MOD_INT -> (no net)
- U1 pad 38: MOD_A -> ROW1
- U1 pad 39: MOD_B -> ROW0
- U1 pad 40: I2C_SDA -> GND
- U1 pad 41: I2C_SCL -> GND
- U1 pad 8: COL0 -> COL7
- U1 pad 9: COL1 -> COL8
- U3 pad 3: +3V3 -> VBUS
- U3 pad 4: +3V3 -> (no net)
- U3 pad 5: VBUS -> +3V3
Routing:
- net ROW5: track 0.00 -> 457.7 mm, vias 0 -> 4
- net ROW3: track 0.00 -> 389.1 mm, vias 0 -> 2
- net ROW4: track 0.00 -> 382.6 mm, vias 0 -> 2
- net ROW1: track 0.00 -> 375.3 mm, vias 0 -> 4
- net ROW2: track 0.00 -> 370.3 mm, vias 0 -> 2
- net COL0: track 0.00 -> 303.0 mm, vias 0 -> 1
- net ROW0: track 0.00 -> 296.8 mm, vias 0 -> 2
- net COL1: track 0.00 -> 294.7 mm, vias 0 -> 1
- net COL2: track 0.00 -> 276.6 mm, vias 0 -> 1
- net COL13: track 0.00 -> 264.7 mm, vias 0 -> 1
- net COL15: track 0.00 -> 246.1 mm, vias 0 -> 1
- net COL3: track 0.00 -> 234.4 mm, vias 0 -> 3
- net COL6: track 0.00 -> 218.1 mm, vias 0 -> 1
- net COL14: track 0.00 -> 216.0 mm, vias 0 -> 3
- net COL4: track 0.00 -> 213.8 mm, vias 0 -> 1
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- added copper zone on B.Cu, net GND
- added copper zone on F.Cu, net GND
Other:
- board size 346.6 x 137.1 mm -> 337.1 x 150.1 mm
- board text added: "OSO75 rev A 2026-06"
